Commit message: Use dummy world link

File: iiwa_description/urdf/iiwa7_aruco.urdf.xacro (robot description, xacro)
@@ -14,19 +14,5 @@
   If you don't want to have that you can define a basic world link (see commented lines)
   -->
-  <!--     <link name="world"/> -->
-  <link name="world">
-    <visual>
-      <origin xyz="0 0 0.42" rpy="0 0 0"/>
-      <geometry>
-	<box size="0.68 0.605 0.84"/>
-      </geometry>
-    </visual>
-    <collision>
-      <origin xyz="0 0 0.42" rpy="0 0 0"/>
-      <geometry>
-	<box size="0.68 0.605 0.84"/>
-      </geometry>
-    </collision>
-  </link>
+  <link name="world"/>
   <gazebo reference="world">
     <static>true</static>
@@ -34,5 +20,5 @@
   <!-- Here we insert an iiwa7 robot in the scene, it's origin is just on top of the box previously defined. You can use 0,0,0 if you don't have that. -->
   <xacro:iiwa7 hardware_interface="$(arg hardware_interface)" robot_name="$(arg robot_name)" parent="world">
-    <origin xyz="0 0 0.84" rpy="0 0 0"/>
+    <origin xyz="0 0 0" rpy="0 0 0"/>
   </xacro:iiwa7>
   <!-- Tool properties -->

Commit message: Configure aruco board with dae on end effector

File: iiwa_description/urdf/iiwa7_aruco.urdf.xacro (robot description, xacro)
@@ -24,5 +24,5 @@
   <!-- Tool properties -->
   <xacro:property name="tool_mass" value="0.200" />
-  <xacro:property name="tool_joint_offset" value="0.00 0.00 0.00" />
+  <xacro:property name="tool_joint_offset" value="0.00 0.00 0.10" />
   <xacro:property name="tool_link_offset" value="0.00 0.00 0.1275" />
   <!--  Here we define a dummy joint between the tip of the iiwa7 and the base of the tool.
@@ -39,16 +39,15 @@
       <origin xyz="0 0 0" rpy="0 0 0"/>
       <geometry>
-	<mesh filename="package://iiwa_description/meshes/iiwa7_aruco/visual/tool.stl"/>
-	<!-- 	<cylinder length="0.1275" radius="0.020"/> -->
+        <!-- Replace with thin box to represent ArUco board -->
+        <!-- <box size="0.40 0.30 0.005"/> 40 cm x 30 cm x 5 mm -->
+        <mesh filename="package://hand_eye_calibration/assets/aruco_board.dae"/>
       </geometry>
-      <material name="Grey"/>
     </visual>
     <collision>
       <origin xyz="0 0 0" rpy="0 0 0"/>
       <geometry>
-	<mesh filename="package://iiwa_description/meshes/iiwa7_aruco/visual/tool.stl"/>
-	<!-- 	<cylinder length="0.1275" radius="0.020"/> -->
+        <!-- Thin box for collision representation -->
+        <box size="0.40 0.30 0.005"/>
       </geometry>
-      <material name="Grey"/>
     </collision>
   </link>

Commit message: Add camera in gazebo

File: iiwa_description/urdf/iiwa7_aruco.urdf.xacro (robot description, xacro)
@@ -60,3 +60,61 @@
   <!--  The TCP frame is here defined -->
   <link name="tool_link_ee"/>
+  <!-- attach a camera frame -->
+  <link name="base_camera_link">
+    <visual>
+      <origin xyz="0 0 0" rpy="0 0 0" />
+      <geometry>
+        <box size="0.1 0.03 0.01" />
+      </geometry>
+      <material name="cam_color">
+        <color rgba="0. 1. 0. 0.3" />
+      </material>
+    </visual>
+    <inertial>
+      <origin xyz="0 0 0" rpy="0 0 0" />
+      <mass value="0.01" />
+      <inertia ixx="0.1" ixy="0.0" ixz="0.0" iyy="0.1" iyz="0.0" izz="0.1" />
+    </inertial>
+  </link>
+  <joint name="camera_joint" type="fixed">
+    <parent link="world" />
+    <child link="base_camera_link" />
+    <origin xyz="0.5 0 0" rpy="${pi/2} -${pi/2} 0" />
+  </joint>
+  <gazebo reference="base_camera_link">
+    <sensor type="camera" name="base_camera">
+      <update_rate>10.0</update_rate>
+      <camera name="camera">
+        <horizontal_fov>1.396</horizontal_fov>
+        <image>
+          <width>640</width>
+          <height>480</height>
+          <format>R8G8B8</format>
+        </image>
+        <clip>
+          <near>0.02</near>
+          <far>30</far>
+        </clip>
+        <noise>
+          <type>gaussian</type>
+          <mean>0.0</mean>
+          <stddev>0.007</stddev>
+        </noise>
+      </camera>
+      <plugin name="camera_controller" filename="libgazebo_ros_camera.so">
+        <alwaysOn>true</alwaysOn>
+        <updateRate>0.0</updateRate>
+        <cameraName>iiwa_base/camera</cameraName>
+        <imageTopicName>image_raw</imageTopicName>
+        <cameraInfoTopicName>camera_info</cameraInfoTopicName>
+        <frameName>camera_link</frameName>
+        <hackBaseline>0.07</hackBaseline>
+        <distortionK1>0.0</distortionK1>
+        <distortionK2>0.0</distortionK2>
+        <distortionK3>0.0</distortionK3>
+        <distortionT1>0.0</distortionT1>
+        <distortionT2>0.0</distortionT2>
+      </plugin>
+    </sensor>
+  </gazebo>
 </robot>

Commit message: Adjust camera pose

File: iiwa_description/urdf/iiwa7_aruco.urdf.xacro (robot description, xacro)
@@ -80,5 +80,5 @@
     <parent link="world" />
     <child link="base_camera_link" />
-    <origin xyz="0.5 0 0" rpy="${pi/2} -${pi/2} 0" />
+    <origin xyz="0.8 0 1.0" rpy="${pi} ${pi} 0" />
   </joint>
   <gazebo reference="base_camera_link">

Commit message: Update pose of aruco board

File: iiwa_description/urdf/iiwa7_aruco.urdf.xacro (robot description, xacro)
@@ -25,5 +25,5 @@
   <xacro:property name="tool_mass" value="0.200" />
   <xacro:property name="tool_joint_offset" value="0.00 0.00 0.10" />
-  <xacro:property name="tool_link_offset" value="0.00 0.00 0.1275" />
+  <xacro:property name="tool_link_offset" value="0.20 0.15 0.00" />
   <!--  Here we define a dummy joint between the tip of the iiwa7 and the base of the tool.
   There is no offset between the two, that means the tool is attached at the robot flange. -->
@@ -56,5 +56,5 @@
     <parent link="tool_link" />
     <child link = "tool_link_ee" />
-    <origin xyz="${tool_link_offset}" rpy="0 0 0" />
+    <origin xyz="${tool_link_offset}" rpy="0 0 ${pi}" />
   </joint>
   <!--  The TCP frame is here defined -->

Commit message: Add camera optical frame
Camera link frame is inconsistent with opencv image coordinate system

File: iiwa_description/urdf/iiwa7_aruco.urdf.xacro (robot description, xacro)
@@ -82,4 +82,19 @@
     <origin xyz="0.8 0 1.0" rpy="${pi} ${pi} 0" />
   </joint>
+  <!-- generate an optical frame
+      http://www.ros.org/reps/rep-0103.html#suffix-frames
+      so that ros and opencv can operate on the camera frame correctly
+      see https://robotics.stackexchange.com/questions/73459/gazebo-camera-frame-is-inconsistent-with-rviz-opencv-convention
+      -->
+  <joint name="camera_optical_joint" type="fixed">
+    <!-- these values have to be these values otherwise the gazebo camera
+        image won't be aligned properly with the frame it is supposedly
+        originating from -->
+    <origin xyz="0 0 0" rpy="${-pi/2} 0 ${-pi/2}"/>
+    <parent link="base_camera_link"/>
+    <child link="base_camera_link_optical"/>
+  </joint>
+  <link name="base_camera_link_optical">
+  </link>
   <gazebo reference="base_camera_link">
     <sensor type="camera" name="base_camera">
@@ -108,5 +123,5 @@
         <imageTopicName>image_raw</imageTopicName>
         <cameraInfoTopicName>camera_info</cameraInfoTopicName>
-        <frameName>camera_link</frameName>
+        <frameName>base_camera_link_optical</frameName>
         <hackBaseline>0.07</hackBaseline>
         <distortionK1>0.0</distortionK1>
